File: kicad/CPU.kicad_sch (KiCad schematic)
At the start: 88 parts, among them U7 MCIMX6Y2CVM08AB, U8 UM803RS, Y1 24 MHz, Y2 32.768 KHz

Commit message: Fix hardware bugs - Fix part number in bom for resistors R103, R113, R114, R118 -> 680K - Fix part number in BOM for resistors R13, R16 -> 68K - Fix part number in BOM for resistor R14 -> 4.7K - Fix part number in BOM for capacitors C100, C101, C12, C13, C130, C131, C133, C135, C140, C141, C15, C19, C57, C58, C7, C99 -> 100nF - Fix footprint for USB-A connectors - Fix power buttom pull-up resistor connection -> connect to +3.3V_STAND_BY
Parts:
- C57, C58: symbol -- database:Capacitors/CAP_0402-100n-50V-X7R-10% -> ts_database:Capacitors/CAP_0402-100n-50V-X7R-10%; LCSC C1523 -> C77020
Connections:
- net +3V3_DCDC: no longer R23.1, R24.1
- net +3V3_STAND_BY: now also R23.1, R24.1
