File: kicad/LCD.kicad_sch (KiCad schematic)
At the start: 82 parts, among them J6 8.15A0.060200, Q1 NTR5105PT1G, Q2 SMMBT3904LT1G, U17 MT9700, U18 TPS65150PWPR, U19 LMV321IDBVR

Commit message: Fix hardware bugs - Fix part number in bom for resistors R103, R113, R114, R118 -> 680K - Fix part number in BOM for resistors R13, R16 -> 68K - Fix part number in BOM for resistor R14 -> 4.7K - Fix part number in BOM for capacitors C100, C101, C12, C13, C130, C131, C133, C135, C140, C141, C15, C19, C57, C58, C7, C99 -> 100nF - Fix footprint for USB-A connectors - Fix power buttom pull-up resistor connection -> connect to +3.3V_STAND_BY
Parts:
- C130, C131, C133, C135, C140, C141: symbol -- database:Capacitors/CAP_0402-100n-50V-X7R-10% -> ts_database:Capacitors/CAP_0402-100n-50V-X7R-10%; LCSC C1523 -> C77020
- R103, R113, R114, R118: symbol -- database:Resistors/RES-SMD-0402-680K-1/16W-1% -> ts_database:Resistors/RES-SMD-0402-680K-1/16W-1%; LCSC C25917 -> C163456
